Commit message: v0.1

File: urdf/differential_robot.urdf.xacro (robot description, xacro)
@@ -14,5 +14,5 @@
       <origin xyz="0 0 0" rpy="1.57 0 1.57"/>
       <geometry>
-        <mesh filename="file:///home/hualde/misCosas/ros2_ws/src/robot_description/meshes/base_link.stl" scale="0.0008 0.0008 0.0008"/>
+        <mesh filename="file:///home/hualde/misCosas/ros2_ws/src/robot_gazebo/meshes/base_link.stl" scale="0.0008 0.0008 0.0008"/>
       </geometry>
       <material name="gray">
@@ -23,5 +23,5 @@
       <origin xyz="0 0 0" rpy="1.57 0 1.57"/>
       <geometry>
-        <mesh filename="file:///home/hualde/misCosas/ros2_ws/src/robot_description/meshes/base_link.stl" scale="0.0008 0.0008 0.0008"/>
+        <mesh filename="file:///home/hualde/misCosas/ros2_ws/src/robot_gazebo/meshes/base_link.stl" scale="0.0008 0.0008 0.0008"/>
       </geometry>
     </collision>
